Commit message: fixed urdf file

File: urdf/fusion_13_structure.urdf.xacro (robot description, xacro)
@@ -2,5 +2,5 @@
 <!-- created with Phobos 0.7 -->
   <robot name="car" xmlns:xacro="http://www.ros.org/wiki/xacro">
-    <xacro:arg name="dae_file" default="$(find Project_robotics)/meshes/fusion_13/body.dae"/>
+    <xacro:arg name="dae_file" default="$(find robotics)/meshes/fusion_13/body.dae"/>
     <link name="base_footprint">
     </link>
@@ -21,5 +21,5 @@
         <origin xyz="1.51 -0.03046 0.325149" rpy="1.570796 0 -3.141593"/>
         <geometry>
-          <mesh filename="package://Project_robotics/meshes/body_collision.stl" scale="0.000965 0.001 0.001"/>
+          <mesh filename="package://robotics/meshes/body_collision.stl" scale="0.000965 0.001 0.001"/>
         </geometry>
       </collision>
@@ -48,5 +48,5 @@
         <origin xyz="0 0 0.0385" rpy="-1.570796 -1.570796 0"/>
         <geometry>
-          <mesh filename="package://Project_robotics/meshes/fusion_13/wheel.dae" scale="0.01 0.01 0.01"/>
+          <mesh filename="package://robotics/meshes/fusion_13/wheel.dae" scale="0.01 0.01 0.01"/>
         </geometry>
         <material name="carpaint_002"/>
@@ -68,5 +68,5 @@
         <origin xyz="0 0 -0.043777" rpy="-1.570796 1.570796 0"/>
         <geometry>
-          <mesh filename="package://Project_robotics/meshes/fusion_13/wheel.dae" scale="0.01 0.01 0.01"/>
+          <mesh filename="package://robotics/meshes/fusion_13/wheel.dae" scale="0.01 0.01 0.01"/>
         </geometry>
         <material name="carpaint_002.001"/>
@@ -88,5 +88,5 @@
         <origin xyz="0 0 0.017382" rpy="-1.570796 -1.570796 0"/>
         <geometry>
-          <mesh filename="package://Project_robotics/meshes/fusion_13/wheel.dae" scale="0.01 0.01 0.01"/>
+          <mesh filename="package://robotics/meshes/fusion_13/wheel.dae" scale="0.01 0.01 0.01"/>
         </geometry>
         <material name="carpaint_002.003"/>
@@ -108,5 +108,5 @@
         <origin xyz="0 0 -0.019214" rpy="-1.570796 1.570796 0"/>
         <geometry>
-          <mesh filename="package://Project_robotics/meshes/fusion_13/wheel.dae" scale="0.01 0.01 0.01"/>
+          <mesh filename="package://robotics/meshes/fusion_13/wheel.dae" scale="0.01 0.01 0.01"/>
         </geometry>
         <material name="carpaint_002.002"/>
@@ -240,5 +240,5 @@
     </plugin>
     <plugin name="gazebo_ros_control" filename="libgazebo_ros_control.so">
-      <robotNamespace>/parkingdemo</robotNamespace>
+      <robotNamespace>/car</robotNamespace>
     </plugin>
   </gazebo>
