Commit message: addded lidar to the urdf

File: urdf/car_model.urdf.xacro (robot description, xacro)
@@ -119,4 +119,23 @@
       </collision>
     </link>
+    <link name="laser">
+      <collision>
+        <origin xyz="0 0 0" rpy="1.5707 0 4.71"/>
+        <geometry>
+          <mesh filename="package://robotics/meshes/rplidar.dae" scale="0.001 0.001 0.001" />
+        </geometry>
+      </collision>
+      <visual>
+        <origin xyz="0 0 0" rpy="1.5707 0 4.71"/>
+        <geometry>
+          <mesh filename="package://robotics/meshes/rplidar.dae" scale="0.001 0.001 0.001" />
+        </geometry>
+      </visual>
+      <inertial>
+        <mass value="1e-5" />
+        <origin xyz="0 0 0" rpy="1.5707 0 4.71"/>
+        <inertia ixx="0" ixy="0" ixz="0" iyy="0" iyz="0" izz="0" />
+      </inertial>
+    </link>
     <joint name="base_link" type="fixed">
       <origin xyz="0 0 0.33" rpy="0 0 0"/>
@@ -165,4 +184,10 @@
       <axis xyz="0 0 1.0"/>
       <limit effort="5000.0" velocity="22.0"/>
+    </joint>
+    <joint name="rplidar_joint" type="fixed">
+      <axis xyz="0 1 0" />
+      <origin xyz="3 0 0.7" rpy="0 0 3.14"/>
+      <parent link="base_link"/>
+      <child link="laser"/>
     </joint>
   <!-- Transmission Tags -->

Commit message: working 2d lidar with slamming(sort off)

File: urdf/car_model.urdf.xacro (robot description, xacro)
@@ -187,5 +187,5 @@
     <joint name="rplidar_joint" type="fixed">
       <axis xyz="0 1 0" />
-      <origin xyz="3 0 0.7" rpy="0 0 3.14"/>
+      <origin xyz="3 0 0.65" rpy="0 0 3.14"/>
       <parent link="base_link"/>
       <child link="laser"/>
@@ -252,5 +252,36 @@
     </actuator>
   </transmission>
-  <!-- Plugin Definitions -->
+    <!-- RpLidar A2 using CPU -->
+    <gazebo reference="laser">
+      <sensor type="ray" name="head_rplidar_sensor">
+        <pose>0 0 0.06 0 0 0</pose>
+        <visualize>false</visualize>
+        <update_rate>40</update_rate>
+        <ray>
+          <scan>
+            <horizontal>
+              <samples>720</samples>
+              <resolution>1</resolution>
+              <min_angle>-3.14159265</min_angle>
+              <max_angle>3.14159265</max_angle>
+            </horizontal>
+          </scan>
+          <range>
+            <min>0.2</min>
+            <max>12.0</max>
+            <resolution>0.01</resolution>
+          </range>
+          <noise>
+            <type>gaussian</type>
+            <mean>0.0</mean>
+            <stddev>0.01</stddev>
+          </noise>
+        </ray>
+        <plugin name="gazebo_ros_head_rplidar_controller" filename="libgazebo_ros_laser.so">
+          <topicName>car/laser/scan</topicName>
+          <frameName>laser</frameName>
+        </plugin>
+      </sensor>
+    </gazebo>
   <gazebo>
     <plugin name="p3d_base_controller" filename="libgazebo_ros_p3d.so">

Commit message: placing the lidar in a position so it doesn't scan the car

File: urdf/car_model.urdf.xacro (robot description, xacro)
@@ -187,5 +187,5 @@
     <joint name="rplidar_joint" type="fixed">
       <axis xyz="0 1 0" />
-      <origin xyz="3 0 0.65" rpy="0 0 3.14"/>
+      <origin xyz="1 0 1.15" rpy="0 0 3.14"/>
       <parent link="base_link"/>
       <child link="laser"/>
